Commit message: cfg and launch
added cfg and launch,
launch doesn't work yet

File: src/BobertLimits/urdf/BobertLimits.urdf (robot description, URDF)
Before this commit: robot BobertClamp, 7 links, 6 joints
Links:
- link End_Effector_Link: geometry collision mesh filename=package://BobertLimits/meshes/End_Effector_Link.STL; visual mesh filename=package://BobertLimits/meshes/End_Effector_Link.STL
- link Servo_Link_1: geometry collision mesh filename=package://BobertLimits/meshes/Servo_Link_1.STL; visual mesh filename=package://BobertLimits/meshes/Servo_Link_1.STL
- link Servo_Link_2: geometry collision mesh filename=package://BobertLimits/meshes/Servo_Link_2.STL; visual mesh filename=package://BobertLimits/meshes/Servo_Link_2.STL
- link Servo_Link_3: geometry collision mesh filename=package://BobertLimits/meshes/Servo_Link_3.STL; visual mesh filename=package://BobertLimits/meshes/Servo_Link_3.STL
- link Servo_Link_4: geometry collision mesh filename=package://BobertLimits/meshes/Servo_Link_4.STL; visual mesh filename=package://BobertLimits/meshes/Servo_Link_4.STL
- link Servo_Link_5: geometry collision mesh filename=package://BobertLimits/meshes/Servo_Link_5.STL; visual mesh filename=package://BobertLimits/meshes/Servo_Link_5.STL
- link base_link: geometry collision mesh filename=package://BobertLimits/meshes/base_link.STL; visual mesh filename=package://BobertLimits/meshes/base_link.STL
Joints:
- joint End_Effector_Joint: limit lower=0 upper=0 effort=0 velocity=0 -> lower=-1.57 upper=1.57 effort=0 velocity=0; origin xyz=-0.0127 0 -0.0455485642329056 rpy=0 0.458786615265371 0 -> xyz=-0.0127 0 -0.045549 rpy=0 0.45879 0
- joint Servo_Joint_1: limit lower=0 upper=0 effort=0 velocity=0 -> lower=-1.57 upper=1.57 effort=0 velocity=0; origin xyz=0.045 0.055 0.098 rpy=1.5707963267949 0 1.89015420534387 -> xyz=0.045 0.055 0.098 rpy=1.5708 0 1.8902
- joint Servo_Joint_2: limit lower=0 upper=0 effort=0 velocity=0 -> lower=-1.57 upper=1.57 effort=0 velocity=0; origin xyz=0 0.0125 0 rpy=1.5707963267949 0 0.980263921832072 -> xyz=0 0.0125 0 rpy=1.5708 0 0.98026
- joint Servo_Joint_3: limit lower=0 upper=0 effort=0 velocity=0 -> lower=-1.57 upper=1.57 effort=0 velocity=0; origin xyz=0.105 0 0 rpy=-3.14159265358979 -0.852180438694167 0 -> xyz=0.105 0 0 rpy=-3.1416 -0.85218 0
- joint Servo_Joint_4: limit lower=0 upper=0 effort=0 velocity=0 -> lower=-1.57 upper=1.57 effort=0 velocity=0; origin xyz=0.0969999999999999 0 0 rpy=-3.14159265358979 -0.158151274017002 0 -> xyz=0.097 0 0 rpy=-3.1416 -0.15815 0
- joint Servo_Joint_5: limit lower=0 upper=0 effort=0 velocity=0 -> lower=-1.57 upper=1.57 effort=0 velocity=0; origin xyz=0.0300514357670951 0 0.0125000000000007 rpy=-1.5707963267949 0.0774701937986736 1.5707963267949 -> xyz=0.030051 0 0.0125 rpy=-1.5708 0.07747 1.5708
